File: hardware/flood_node_pcb/EIN_Flood_Node.kicad_sch (KiCad schematic)
At the start: 6 parts, among them J1 SOLAR_IN_12V, J2 BATTERY_LiFePO4, J3 JSN-SR04T_ULTRASONIC, J4 RAIN_GAUGE_PULSE, U1 ESP32-S3-WROOM-1, U2 SX1276_LoRa

Commit message: Fix KiCanvas white screen: remove unsupported comments in PCB and align schematic syntax
Parts:
- added D1: SMAJ18A, symbol Device:D_TVS
- added D2: ESD5Z3.3, symbol Device:D_TVS
- added D3: PWR_GREEN, symbol Device:LED
- added D4: STAT_BLUE, symbol Device:LED
- added D5: ALERT_RED, symbol Device:LED
- added J6: SMA_ANTENNA, symbol Connector:SMA
- added R3: 2.2k, symbol Device:R
- added R4: 3.3k, symbol Device:R
- added R5: 10k, symbol Device:R
- added SW1: RESET_SW, symbol Switch:SW_Push
- added U3: SHT31_ENV, symbol Sensor:SHT31
- added U4: DS3231_RTC, symbol Sensor:DS3231
- added U5: ADS1115_ADC, symbol Sensor:ADS1115
- added U6: BQ24650_MPPT, symbol Power:BQ24650
- added U7: AP2112K_3.3V, symbol Power:AP2112K
- added U8: TPS61023_5V, symbol Power:TPS61023
- J1: value SOLAR_IN_12V -> SOLAR_IN; footprint TerminalBlock:TerminalBlock_bornier-2_P5.08mm -> (none)
- J2: value BATTERY_LiFePO4 -> LIFEPO4_3.2V; footprint TerminalBlock:TerminalBlock_bornier-2_P5.08mm -> (none)
- J3: value JSN-SR04T_ULTRASONIC -> JSN-SR04T; footprint TerminalBlock:TerminalBlock_bornier-4_P3.81mm -> (none)
- J4: value RAIN_GAUGE_PULSE -> RAIN_GAUGE; footprint TerminalBlock:TerminalBlock_bornier-2_P3.81mm -> (none)
- U1: footprint RF_Module:ESP32-S3-WROOM-1 -> (none)
- U2: value SX1276_LoRa -> SX1276_868MHz; footprint RF_Module:Ai-Thinker_Ra-02 -> (none)
Connections:
- net +5V: now reaches J3.1 (Pin_1)
- net +5V: now also U8.6 (VOUT)
- net JSN_TRIG: now reaches J3.2 (Pin_2)
- net JSN_TRIG: now also U1.5 (IO5_JSN_TRIG)
- net at J3.3 (Pin_3): now also R3.1
- net GND: now reaches J3.4 (Pin_4)
- net GND: now also J1.2 (Pin_2), J2.2 (Pin_2), J4.2 (Pin_2), U1.0 (GND_THERMAL), U1.1 (GND), U2.2 (GND), J6.2 (GND), R4.2, U3.8 (VSS), U4.13 (GND), U6.16 (GND), U7.2 (GND), U8.3 (GND)
- net RAIN_IRQ: now reaches J4.1 (Pin_1)
- net RAIN_IRQ: now also U1.4 (IO4_RAIN), D2.1 (A), R5.1
- net LORA_DIO0: now reaches U1.10 (IO11_MOSI)
- net LORA_DIO0: now also U1.14 (IO21_LORA_DIO0), U2.14 (DIO0), U2.5 (MOSI)
- net SPI_SCK: now reaches U1.11 (IO12_SCK)
- net SPI_SCK: now also U2.4 (SCK)
- net SPI_MISO: now reaches U1.12 (IO13_MISO)
- net SPI_MISO: now also U2.6 (MISO)
- net LORA_RESET: now reaches U1.13 (IO14_LORA_RST)
- net LORA_RESET: now also U2.9 (NRESET)
- net +3.3V: now reaches U1.2 (3V3)
- net +3.3V: now also U2.1 (VCC), R5.2, U3.5 (VDD), U4.2 (VCC), U7.5 (VOUT)
- net VBAT_SENSE: now reaches U1.21 (IO1_ADC_BATT)
- net MCU_RESET: now reaches U1.3 (EN)
- net MCU_RESET: now also SW1.1
- net DEBUG_TXD: now reaches U1.43 (TXD0)
- net DEBUG_RXD: now reaches U1.44 (RXD0)
- net JSN_ECHO: now reaches U1.6 (IO6_JSN_ECHO)
- net JSN_ECHO: now also R3.2, R4.1
- net I2C_SDA: now reaches U1.7 (IO8_I2C_SDA)
- net I2C_SDA: now also U3.1 (SDA), U4.15 (SDA), U5.5 (SDA)
- net I2C_SCL: now reaches U1.8 (IO9_I2C_SCL)
- net I2C_SCL: now also U3.4 (SCL), U4.16 (SCL), U5.8 (SCL)
- net LORA_NSS: now reaches U1.9 (IO10_LORA_CS)
- net LORA_NSS: now also U2.3 (NSS)
- net SOLAR_VIN: now reaches J1.1 (Pin_1)
- net SOLAR_VIN: now also U5.2 (A1), U6.1 (VCC)
- net VBAT: now reaches J2.1 (Pin_1)
- net VBAT: now also U5.1 (A0), U6.12 (VBAT), U7.1 (VIN), U7.3 (EN), U8.1 (VIN)
- new net: J6.1 (SIG), U2.16 (PA_BOOST)
Other:
- note added: "1. POWER: SOLAR MPPT BQ24650 + 3.2V LiFePO4 + 3.3V LDO & 5V BOOST"
- note added: "2. CORE MCU: ESP32-S3 (EDGE AI ENGINE, TFLITE MICRO, POWER GATING)"
- note added: "3. RF: SEMTECH SX1276 LORA (865-867MHz IN865) + 50 OHM SMA BULKHEAD"
- note added: "4. SENSOR TRANSDUCERS (JSN-SR04T ULTRASONIC & TIPPING RAIN GAUGE)"
- note added: "5. I2C CLUSTER (SHT31 TEMP/RH, DS3231 RTC, ADS1115 16-BIT ADC)"
- note removed: "CORE & RF: ESP32-S3 (TFLite Micro) <SPI> Semtech SX1276 LoRa (865-867 MHz)"
- note removed: "I2C BUS: SHT31 (0x44) | DS3231 RTC (0x68) | ADS1115 ADC (0x48)"
- note removed: "POWER SUBSYSTEM: MPPT BQ24650 -> 3.3V LDO AP2112K + 5V BOOST TPS61023 + LOAD SWITCH TPS22919"

Commit message: adding some details of team
Other:
- title: EIN Flagship Flood / Water-Level Node - Production Hardware -> SWARNIM Flagship Flood / Water-Level Node - Production Hardware
Changed lines of the file:
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@@
   (paper "A3")
   (title_block
-    (title "EIN Flagship Flood / Water-Level Node - Production Hardware")
-    (date "2026-09-05")
+    (title "SWARNIM Flagship Flood / Water-Level Node - Production Hardware")
+    (date "2026-09-09")
     (rev "v1.0-RC1")
     (company "Team Swarnim | SIH 2026 Problem Statement 26178 (Qualcomm Inc.)")
-    (comment 1 "Dual-Tier Edge AI & Resilient LoRa Sensing Node")
+    (comment 1 "Tier 1 Low-Cost Sensing Node (Feeds Tier 2 Raspberry Pi 5 Hub)")
     (comment 2 "MCU: ESP32-S3 | RF: SX1276 (865-867MHz) | Solar MPPT: BQ24650")
     (comment 3 "Sensors: JSN-SR04T Ultrasonic + Rain Gauge + SHT31 + DS3231 + ADS1115")
